File: circuit/museon.kicad_pcb (KiCad board)
At the start: 2 copper layers, 90 x 70 mm, 13 parts, among them J1 Conn_01x04_MountingPin, J2 Conn_01x04_MountingPin, J3 Conn_01x04_MountingPin, J4 Conn_01x04_MountingPin, J5 Conn_01x04_MountingPin, J6 Conn_01x04_MountingPin, J7 Conn_01x04_MountingPin, J8 Conn_01x04_MountingPin, J9 Conn_01x04_MountingPin

Commit message: update
Parts:
- added REF**: MountingHole_3.2mm_M3, MountingHole:MountingHole_3.2mm_M3, F.Cu at (97.0, 73.0)
- added REF**: MountingHole_3.2mm_M3, MountingHole:MountingHole_3.2mm_M3, F.Cu at (17.0, 73.0)
- added REF**: MountingHole_3.2mm_M3, MountingHole:MountingHole_3.2mm_M3, F.Cu at (97.0, 133.0)
- moved JSC1 10.0 mm to (38.0, 75.0)
- moved R2 5.70 mm to (24.1, 87.8), turned to 90 degrees
- moved R1 2.47 mm to (28.0, 87.8), turned to 90 degrees
Routing:
- net Net-(A1-GPIO20): track 30.2 -> 21.8 mm
- net Net-(A1-GPIO21): track 30.1 -> 21.8 mm
- net Net-(J1-Pin_3): track 226.4 -> 232.5 mm
- net Net-(A1-3V3): track 13.7 -> 8.09 mm
- net Net-(JSC1-Pin_4): track 11.4 -> 6.23 mm
